File: ejemplos/KiCad/src/555_PCB/001.sch (KiCad schematic (older format))
At the start: 13 parts, among them U1 LM555

Commit message: Auto stash before merge of "master" and "origin/master"
Parts:
- removed U1, U?: LM555, symbol linear:LM555
- added U1, U2: NE555, Wickerlib:SOIC-8-3.9x4.9MM-P1.27MM, symbol 555_Semaforo:NE555
- C1, C2: footprint (none) -> Capacitor_SMD:C_1206_3216Metric_Pad1.39x1.80mm_HandSolder
- R1, R2, R3: footprint Resistor_SMD:R_1206_3216Metric_Pad1.42x1.75mm_HandSolder -> Resistor_SMD:R_1206_3216Metric_Pad1.39x1.80mm_HandSolder
- R4: value 330 -> 470; footprint Resistor_SMD:R_1206_3216Metric_Pad1.42x1.75mm_HandSolder -> Resistor_SMD:R_1206_3216Metric_Pad1.39x1.80mm_HandSolder
- R5: value 330 -> 47k; footprint Resistor_SMD:R_1206_3216Metric_Pad1.42x1.75mm_HandSolder -> Resistor_SMD:R_1206_3216Metric_Pad1.39x1.80mm_HandSolder
Connections:
- net labels added: +12V
- wire segments 27 -> 58
- no-connect marks 2 -> 3
Other:
- moved on the sheet: C1, C2, D2, D3, E1, R3, R4, R5
