File: ejemplos/KiCad/src/Universal/10mm4Pins/001.kicad_pcb (KiCad board)
At the start: 2 copper layers, 37.2 x 73.4 mm, 13 parts, among them J1 CONN_01X04

Commit message: Some updates
Parts:
- added G***: LOGO, HG_OshPark:OSHpark-1-1100, B.Cu at (134.2, 76.2)
- added G***: LOGO, HG_OshPark:OSHpark-2-1800, B.Cu at (133.8, 80.6)
