File: ejemplos/KiCad/src/Universal/5mm4Pins/001.kicad_pcb (KiCad board)
At the start: 2 copper layers, 37.2 x 73.4 mm, 15 parts, among them J1 CONN_01X04

Commit message: Some updates
Parts:
- D1, D2, D3: footprint Semaforo:LED_D10.0mm -> Semaforo:LED_D5.0mm
- E1: footprint Semaforo:10mm.All.01 -> Semaforo:5mm.All.01
- moved svg2mod 35.2 mm to (167.0, 119.4)
- moved svg2mod 35.2 mm to (167.0, 121.3)
- moved REF** 16.8 mm to (150.5, 114.9)
- moved G*** 12.3 mm to (121.9, 77.5)
- moved G*** 12.1 mm to (123.2, 71.1)
- moved E1 10.2 mm to (134.0, 99.1)
Routing:
- net Net-(D1-Pad2): track 65.1 -> 0.00 mm
- net Net-(D2-Pad2): track 50.2 -> 0.00 mm
- net Net-(D3-Pad2): track 36.6 -> 0.00 mm
- net Net-(D1-Pad1): track 4.70 -> 0.00 mm
- net Net-(D2-Pad1): track 4.68 -> 0.00 mm
- net Net-(D3-Pad1): track 4.63 -> 0.00 mm
Other:
- board size 37.2 x 73.4 mm -> 22.8 x 45 mm
